Commit message: Completed assignment

File: my_robot/urdf/my_robot.xacro (robot description, xacro)
@@ -22,5 +22,5 @@
             <origin xyz="0 0 0" rpy=" 0 0 0"/>
             <geometry>
-                <box size=".4 .2 .1"/>
+                <box size=".6 .2 .1"/>
             </geometry>
         </collision>
@@ -28,5 +28,5 @@
             <origin xyz="0 0 0" rpy=" 0 0 0"/>
             <geometry>
-                <box size=".4 .2 .1"/>
+                <box size=".6 .2 .1"/>
             </geometry>
         </visual>
@@ -142,5 +142,5 @@
 	</link>
     <joint type="fixed" name="camera_joint">
-        <origin xyz="0.2 0 0" rpy="0 0 0"/>
+        <origin xyz="0.3 0 0" rpy="0 0 0"/>
         <child link="camera"/>
         <parent link="chassis"/>
@@ -171,5 +171,5 @@
     </link>
     <joint type="fixed" name="hokuyo_joint">
-        <origin xyz="0.15 0 0.1" rpy="0 0 0"/>
+        <origin xyz="0.25 0 0.1" rpy="0 0 0"/>
         <child link="hokuyo"/>
         <parent link="chassis"/>
@@ -177,14 +177,14 @@
     </joint>
 	<gazebo reference="left_wheel">
-		<material>Gazebo/Green</material>
+		<material>Gazebo/Gray</material>
 	</gazebo>
 	<gazebo reference="right_wheel">
-		<material>Gazebo/Green</material>
+		<material>Gazebo/Gray</material>
 	</gazebo>
 	<gazebo reference="chassis">
+		<material>Gazebo/Purple</material>
+	</gazebo>
+	<gazebo reference="camera">
 		<material>Gazebo/Blue</material>
 	</gazebo>
-	<gazebo reference="camera">
-		<material>Gazebo/Red</material>
-	</gazebo>
 </robot>
